File: PCB/WaveTheory.kicad_pcb (KiCad board)
At the start: 2 copper layers, 284.6 x 93.7 mm, 151 parts, among them J2 USB_C_Receptacle_USB2.0, J3 Battery, J4 Conn_01x04, J6 TC2030_SWD, Q1 AO3401A, SW1 SW_SPDT, SW2 SW_Push, SW3 RotaryEncoder_Switch_MP, SW4 RotaryEncoder_Switch_MP, SW5 RotaryEncoder_Switch_MP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

Commit message: First revision
Changed lines of the file:
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@@
 		(fp_circle
 			(center 0 0)
-			(end 0 -2)
+			(end 0.000001 -2)
 			(stroke
 				(width 0.12)
@@
 		)
 		(pad "B" thru_hole circle
-			(at 2.499999 7.499997 328)
+			(at 2.5 7.499997 328)
 			(size 2 2)
 			(drill 1)
@@
 	(segment
 		(start 139.149686 30.113442)
-		(end 139.149686 22.812645)
+		(end 139.149686 23.812645)
 		(width 0.5)
 		(layer "F.Cu")
@@
 	)
 	(segment
-		(start 139.149686 22.812645)
+		(start 140.149686 22.812645)
 		(end 141.121487 22.812645)
 		(width 0.5)
@@
 		(width 0.5)
 		(layer "F.Cu")
+		(net 4)
+	)
+	(arc
+		(start 140.149686 22.812645)
+		(mid 139.442579 23.105538)
+		(end 139.149686 23.812645)
+		(width 0.5)
+		(layer "F.Cu")
